Commit message: Add serial

File: robot_description/youbot.urdf (robot description, URDF)
Before this commit: robot youbot, 10 links, 9 joints
Joints:
- joint arm_joint_0: origin xyz=0.143 0 0.046 rpy=0 0 0 -> xyz=0 0 0 rpy=0 0 0
- joint arm_joint_1: axis 0 0 1 -> 0 0 -1; origin xyz=0.024 0 0.096 rpy=0 0 0 -> xyz=0.024 0 0.096 rpy=0 0 2.96705
- joint arm_joint_2: axis 0 -1 0 -> 0 1 0; origin xyz=0.033 0 0.019 rpy=0 0 0 -> xyz=0.033 0 0.019 rpy=0 -1.1344640 0
- joint arm_joint_3: origin xyz=0.000 0.000 0.155 rpy=0 0 0 -> xyz=0.000 0.000 0.155 rpy=0 2.54818 0
- joint arm_joint_4: axis 0 -1 0 -> 0 1 0; origin xyz=0.000 0.000 0.135 rpy=0 0 0 -> xyz=0.000 0.000 0.135 rpy=0 -1.7889624 0
- joint arm_joint_5: axis 0 0 1 -> 0 0 -1; origin xyz=-0.002 0 0.130 rpy=0 0 0 -> xyz=-0.002 0 0.130 rpy=0 0 2.923426497
